File: car.kicad_pcb (KiCad board)
At the start: 2 copper layers, 3 parts, among them SW1 Push_Button

Commit message: add car
Parts:
- removed SW1: Push_Button, PCM_4ms_Switch:Button_PB20B
- added 9V1: MountingHole_M3_3.2mm_Pad, PCM_SL_Mechanical:MountingHole_3.2mm_Pad, F.Cu at (35.0, 59.2)
- added GND1: MountingHole_M3_3.2mm_Pad, PCM_SL_Mechanical:MountingHole_3.2mm_Pad, F.Cu at (34.6, 79.8)
- added J1: ServoPort_01, PCM_SL_Connectors:ServoPort_01_Vertical, F.Cu at (31.8, 34.1)
- added SW2: Push_Button, Button_Switch_THT:SW_PUSH_6mm, F.Cu at (72.9, 34.4)
- added SW3: Slide_Switch_SPDT_P3mm_10x5x10mm, PCM_SL_Devices:Slide_Switch_SPDT_P3mm_10x5x10mm, F.Cu at (34.6, 67.4)
- added m1: MountingHole_M3_3.2mm_Pad, PCM_SL_Mechanical:MountingHole_3.2mm_Pad, F.Cu at (29.2, 87.8)
- added m2: MountingHole_M3_3.2mm_Pad, PCM_SL_Mechanical:MountingHole_3.2mm_Pad, F.Cu at (29.2, 95.3)
Connections:
- A2 pad A0: unconnected-(A2-PadA0) -> Net-(J1-IN1)
- A2 pad GND1: unconnected-(A2-GND-PadGND1) -> Net-(A2-GND-PadGND1)
- A2 pad VIN: unconnected-(A2-PadVIN) -> Net-(CR1-VS)
- CR1 pad 11: unconnected-(CR1-OUTPUT3-Pad11) -> Net-(CR1-OUTPUT3)
- CR1 pad 12: Net-(A2-GND-PadGND2) -> Net-(A2-GND-PadGND1)
- CR1 pad 13: Net-(A2-GND-PadGND2) -> Net-(A2-GND-PadGND1)
- CR1 pad 14: unconnected-(CR1-OUTPUT4-Pad14) -> Net-(CR1-OUTPUT4)
- CR1 pad 4: unconnected-(CR1-GND-Pad4) -> Net-(A2-GND-PadGND2)
- CR1 pad 5: unconnected-(CR1-GND-Pad5) -> Net-(A2-GND-PadGND2)
- CR1 pad 8: unconnected-(CR1-VS-Pad8) -> Net-(CR1-VS)
Routing:
- net Net-(A2-GND-PadGND1): track 0.00 -> 121.8 mm
- net Net-(CR1-VS): track 0.00 -> 93.6 mm
- net Net-(A2-3.3V): track 29.2 -> 69.6 mm
- net Net-(A2-GND-PadGND2): track 43.8 -> 82.0 mm
- net Net-(J1-IN1): track 0.00 -> 27.1 mm
- net Net-(A2-PadD4): track 47.1 -> 20.6 mm
- net Net-(CR1-INPUT4): track 57.2 -> 79.5 mm
- net Net-(CR1-OUTPUT3): track 0.00 -> 21.0 mm
- net Net-(CR1-OUTPUT4): track 0.00 -> 20.9 mm
- net Net-(CR1-INPUT3): track 42.4 -> 33.0 mm
- net Net-(9V1-Pad1): track 0.00 -> 8.37 mm
- net Net-(CR1-VSS): track 41.3 -> 38.8 mm
Other:
- board outline added: 64 x 95.2 mm
- board text added: "9V"
- board text added: "GND"
- board text added: "M1"
- board text added: "M2"
- board text added: "e a sports"
